File: BME688-ML-V1-PCB.kicad_pcb (KiCad board)
At the start: 2 copper layers, 25.4 x 25.4 mm, 29 parts, among them SW1 434133025816, U1 STM32L431KBU6TR, U2 BME688

Commit message: remove dependency on global library
Parts:
- C1, C2, C3, C4, C5, C6, C7: footprint 1GlobalFootprintsLibrary:C_0603_nominal -> 1projectLibrary:C_0603_nominal
- CONN1, CONN2: value SM04B-SRSS-TB(LF)(DN)(P) -> SM04B-SRSS-TB
- R1, R2, R3, R4, R5, R6, R7, R8: footprint 1GlobalFootprintsLibrary:R_0603_nominal -> 1projectLibrary:R_0603_nominal
Connections:
- net Net-(CONN3-CD) renamed CardDetect
